File: hardware/qwiic-obd/iso.kicad_sch (KiCad schematic)
At the start: 20 parts, among them Q701 2N7002, Q702 2N7002, Q703 2N7002, Q704 MMBT3904, U701 NCS20072, U702 SC16IS741A, X701 ASV-12.000MHZ-EJ-T

Commit message: Added initial layout (parts dump)
Parts:
- D701: footprint Package_TO_SOT_SMD:SOT-323_SC-70 -> Diode_SMD:D_SOD-123; symbol Diode:BAT54W -> Diode:BAT54J
Connections:
- net GND: now also D701.2 (A); no longer D701.1 (A)
- net at R707.1, U701.2 (-): now also D701.1 (K); no longer D701.3 (K)
Changed lines of the file:
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@@
     (pin "1")
   )
-  (symbol (lib_id "Diode:BAT54W") (at 77.47 116.84 270) (unit 1)
+  (symbol (lib_id "Diode:BAT54J") (at 77.47 116.84 270) (unit 1)
     (in_bom yes) (on_board yes)
     (property "Reference" "D701" (id 0) (at 80.7466 115.6716 90)
@@
       (effects (font (size 1.27 1.27)) (justify left))
     )
-    (property "Footprint" "Package_TO_SOT_SMD:SOT-323_SC-70" (id 2) (at 73.025 116.84 0)
+    (property "Footprint" "Diode_SMD:D_SOD-123" (id 2) (at 73.025 116.84 0)
       (effects (font (size 1.27 1.27)) hide)
     )
@@
     (pin "1")
     (pin "2")
-    (pin "3")
   )
   (symbol (lib_id "power:GND") (at 109.22 184.15 0) (unit 1)

Commit message: OK, layout v1 complete
Parts:
- removed R710: 10k, Resistor_SMD:R_0805_2012Metric_Pad1.20x1.40mm_HandSolder, symbol Device:R
- renumbered R711 to R710
Changed lines of the file:
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@@
   (junction (at 173.99 115.57) (diameter 0) (color 0 0 0 0)
-  )
-  (junction (at 128.27 170.18) (diameter 0) (color 0 0 0 0)
   )
   (junction (at 218.44 134.62) (diameter 0) (color 0 0 0 0)
@@
     (stroke (width 0) (type default) (color 0 0 0 0))
   )
-  (wire (pts (xy 128.27 135.89) (xy 128.27 138.43))
-    (stroke (width 0) (type default) (color 0 0 0 0))
-  )
   (wire (pts (xy 97.79 109.22) (xy 101.6 109.22))
     (stroke (width 0) (type default) (color 0 0 0 0))
@@
     (stroke (width 0) (type default) (color 0 0 0 0))
   )
-  (wire (pts (xy 128.27 170.18) (xy 121.92 170.18))
-    (stroke (width 0) (type default) (color 0 0 0 0))
-  )
   (wire (pts (xy 50.8 105.41) (xy 50.8 106.68))
     (stroke (width 0) (type default) (color 0 0 0 0))
@@
     (stroke (width 0) (type default) (color 0 0 0 0))
   )
-  (wire (pts (xy 128.27 170.18) (xy 142.24 170.18))
+  (wire (pts (xy 121.92 170.18) (xy 142.24 170.18))
     (stroke (width 0) (type default) (color 0 0 0 0))
   )
@@
   )
   (wire (pts (xy 58.42 180.34) (xy 58.42 184.15))
-    (stroke (width 0) (type default) (color 0 0 0 0))
-  )
-  (wire (pts (xy 128.27 146.05) (xy 128.27 170.18))
     (stroke (width 0) (type default) (color 0 0 0 0))
   )
@@
   (symbol (lib_id "power:+3V3") (at 135.89 135.89 0) (unit 1)
     (in_bom yes) (on_board yes) (fields_autoplaced)
-    (property "Reference" "#PWR0713" (id 0) (at 135.89 139.7 0)
+    (property "Reference" "#PWR0712" (id 0) (at 135.89 139.7 0)
       (effects (font (size 1.27 1.27)) hide)
     )
@@
   (symbol (lib_id "Device:R") (at 135.89 142.24 0) (unit 1)
     (in_bom yes) (on_board yes)
-    (property "Reference" "R711" (id 0) (at 137.668 141.0716 0)
+    (property "Reference" "R710" (id 0) (at 137.668 141.0716 0)
       (effects (font (size 1.27 1.27)) (justify left))
     )
@@
   (symbol (lib_id "power:+3V3") (at 109.22 138.43 0) (unit 1)
     (in_bom yes) (on_board yes) (fields_autoplaced)
-    (property "Reference" "#PWR0714" (id 0) (at 109.22 142.24 0)
+    (property "Reference" "#PWR0713" (id 0) (at 109.22 142.24 0)
       (effects (font (size 1.27 1.27)) hide)
     )
@@
   (symbol (lib_id "power:GND") (at 247.65 149.86 0) (unit 1)
     (in_bom yes) (on_board yes)
-    (property "Reference" "#PWR0717" (id 0) (at 247.65 156.21 0)
+    (property "Reference" "#PWR0716" (id 0) (at 247.65 156.21 0)
       (effects (font (size 1.27 1.27)) hide)
     )
@@
   (symbol (lib_id "power:GND") (at 58.42 184.15 0) (unit 1)
     (in_bom yes) (on_board yes) (fields_autoplaced)
-    (property "Reference" "#PWR0720" (id 0) (at 58.42 190.5 0)
+    (property "Reference" "#PWR0719" (id 0) (at 58.42 190.5 0)
       (effects (font (size 1.27 1.27)) hide)
     )
@@
     (pin "1")
   )
-  (symbol (lib_id "Device:R") (at 128.27 142.24 0) (unit 1)
-    (in_bom yes) (on_board yes)
-    (property "Reference" "R710" (id 0) (at 130.048 141.0716 0)
-      (effects (font (size 1.27 1.27)) (justify left))
-    )
-    (property "Value" "10k" (id 1) (at 130.048 143.383 0)
-      (effects (font (size 1.27 1.27)) (justify left))
-    )
-    (property "Footprint" "Resistor_SMD:R_0805_2012Metric_Pad1.20x1.40mm_HandSolder" (id 2) (at 126.492 142.24 90)
-      (effects (font (size 1.27 1.27)) hide)
-    )
-    (property "Datasheet" "~" (id 3) (at 128.27 142.24 0)
-      (effects (font (size 1.27 1.27)) hide)
-    )
-    (pin "1")
-    (pin "2")
-  )
   (symbol (lib_id "power:GND") (at 218.44 138.938 0) (unit 1)
     (in_bom yes) (on_board yes)
-    (property "Reference" "#PWR0715" (id 0) (at 218.44 145.288 0)
+    (property "Reference" "#PWR0714" (id 0) (at 218.44 145.288 0)
       (effects (font (size 1.27 1.27)) hide)
     )
@@
   (symbol (lib_id "power:+3V3") (at 91.44 143.51 0) (unit 1)
     (in_bom yes) (on_board yes) (fields_autoplaced)
-    (property "Reference" "#PWR0716" (id 0) (at 91.44 147.32 0)
+    (property "Reference" "#PWR0715" (id 0) (at 91.44 147.32 0)
       (effects (font (size 1.27 1.27)) hide)
     )
@@
   (symbol (lib_id "power:+3V3") (at 58.42 161.29 0) (unit 1)
     (in_bom yes) (on_board yes) (fields_autoplaced)
-    (property "Reference" "#PWR0718" (id 0) (at 58.42 165.1 0)
+    (property "Reference" "#PWR0717" (id 0) (at 58.42 165.1 0)
       (effects (font (size 1.27 1.27)) hide)
     )
@@
   (symbol (lib_id "power:GND") (at 87.63 182.88 0) (unit 1)
     (in_bom yes) (on_board yes) (fields_autoplaced)
-    (property "Reference" "#PWR0719" (id 0) (at 87.63 189.23 0)
+    (property "Reference" "#PWR0718" (id 0) (at 87.63 189.23 0)
       (effects (font (size 1.27 1.27)) hide)
     )
@@
     (pin "7")
   )
-  (symbol (lib_id "power:+3V3") (at 128.27 135.89 0) (unit 1)
-    (in_bom yes) (on_board yes) (fields_autoplaced)
-    (property "Reference" "#PWR0712" (id 0) (at 128.27 139.7 0)
-      (effects (font (size 1.27 1.27)) hide)
-    )
-    (property "Value" "+3V3" (id 1) (at 128.27 130.81 0))
-    (property "Footprint" "" (id 2) (at 128.27 135.89 0)
-      (effects (font (size 1.27 1.27)) hide)
-    )
-    (property "Datasheet" "" (id 3) (at 128.27 135.89 0)
-      (effects (font (size 1.27 1.27)) hide)
-    )
-    (pin "1")
-  )
   (symbol (lib_id "Diode:BAT54J") (at 77.47 116.84 270) (unit 1)
     (in_bom yes) (on_board yes)
@@
   (symbol (lib_id "power:GND") (at 109.22 184.15 0) (unit 1)
     (in_bom yes) (on_board yes) (fields_autoplaced)
-    (property "Reference" "#PWR0721" (id 0) (at 109.22 190.5 0)
-      (effects (font (size 1.27 1.27)) hide)
-    )
+    (property "Reference" "#PWR0720" (id 0) (at 109.22 190.5 0)
+      (effects (font (size 1.27 1.27)) hide)
+    )

Commit message: Fix title block
Other:
- title: Vehicle CAN Collector -> QWIIC OBDII Interface
Changed lines of the file:
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@@
   (paper "A4")
   (title_block
-    (title "Vehicle CAN Collector")
-    (date "2022-12-29")
+    (title "QWIIC OBDII Interface")
+    (date "2023-01-03")
     (rev "1")
     (company "Gavin Hurlbut")

Commit message: Shrunk layout a bit
Parts:
- D701: value BAT54W -> BAT54J
- X701: Digikey (none) -> 535-9309-1-ND
Changed lines of the file:
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@@
+      (effects (font (size 1.27 1.27)) hide)
+    )
+    (property "Digikey" "535-9309-1-ND" (id 4) (at 58.42 172.72 0)
       (effects (font (size 1.27 1.27)) hide)
     )
@@
       (effects (font (size 1.27 1.27)) (justify left))
     )
-    (property "Value" "BAT54W" (id 1) (at 80.7466 117.983 90)
-      (effects (font (size 1.27 1.27)) (justify left))
-    )
+    (property "Value" "BAT54J" (id 1) (at 80.7466 117.983 90)
+      (effects (font (size 1.27 1.27)) (justify left))
+    )

Commit message: Switch out the PIC for an ATtiny424.
Parts:
- renumbered C701 to C29, D701 to D20, Q701 to Q18, Q702 to Q19, Q704 to Q20, Q703 to Q21, R704 to R50, R708 to R51, R707 to R52, R701 to R53, R705 to R54, R702 to R55, R710 to R56, R709 to R57, R706 to R58, R703 to R59, U701 to U17, U702 to U18, X701 to X1
