File: hardware/qwiic-obd/qwiic-obd.kicad_sch (KiCad schematic)
At the start: 8 parts, among them J101 I2C_STANDARD, J102 DB15_Female_HighDensity_Mount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, J103 I2C_STANDARD

Commit message: Moved to using shared KiCad libs, regen gerbers
Parts:
- D101, D102, D103, D104, D105: footprint SparkFun-DiscreteSemi:SOT23-3 -> SparkFun-Silicon-Standard:SOT23-3
- J101, J103: value I2C_STANDARD -> QWIIC Connector; footprint UltraLibrarian:PRT-16766 -> Beirdo:QWIIC Connector
Changed lines of the file:
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@@
       (effects (font (size 1.524 1.524)))
     )
-    (property "Footprint" "SparkFun-DiscreteSemi:SOT23-3" (id 2) (at 53.594 131.826 0)
+    (property "Footprint" "SparkFun-Silicon-Standard:SOT23-3" (id 2) (at 53.594 131.826 0)
       (effects (font (size 1.524 1.524)) hide)
     )
@@
       (effects (font (size 1.524 1.524)))
     )
-    (property "Footprint" "SparkFun-DiscreteSemi:SOT23-3" (id 2) (at 53.594 111.506 0)
+    (property "Footprint" "SparkFun-Silicon-Standard:SOT23-3" (id 2) (at 53.594 111.506 0)
       (effects (font (size 1.524 1.524)) hide)
     )
@@
     (property "Reference" "D104" (id 0) (at 53.34 157.353 0))
     (property "Value" "PESD1CAN" (id 1) (at 53.34 159.6644 0))
-    (property "Footprint" "SparkFun-DiscreteSemi:SOT23-3" (id 2) (at 49.022 167.894 0)
+    (property "Footprint" "SparkFun-Silicon-Standard:SOT23-3" (id 2) (at 49.022 167.894 0)
       (effects (font (size 0.508 0.508)) hide)
     )
@@
     (property "Reference" "D103" (id 0) (at 53.086 137.033 90))
     (property "Value" "MMBZ27VCLT1" (id 1) (at 53.086 139.3444 90))
-    (property "Footprint" "SparkFun-DiscreteSemi:SOT23-3" (id 2) (at 55.626 147.066 0)
+    (property "Footprint" "SparkFun-Silicon-Standard:SOT23-3" (id 2) (at 55.626 147.066 0)
       (effects (font (size 0.508 0.508)) hide)
     )
@@
     (property "Reference" "D105" (id 0) (at 53.086 174.879 0))
     (property "Value" "PESD1CAN" (id 1) (at 53.086 177.1904 0))
-    (property "Footprint" "SparkFun-DiscreteSemi:SOT23-3" (id 2) (at 48.768 185.42 0)
+    (property "Footprint" "SparkFun-Silicon-Standard:SOT23-3" (id 2) (at 48.768 185.42 0)
       (effects (font (size 0.508 0.508)) hide)
     )
@@
     (in_bom yes) (on_board yes) (fields_autoplaced)
     (property "Reference" "J103" (id 0) (at 28.575 53.34 0))
-    (property "Value" "I2C_STANDARD" (id 1) (at 28.575 55.88 0))
-    (property "Footprint" "UltraLibrarian:PRT-16766" (id 2) (at 27.432 67.31 0)
+    (property "Value" "QWIIC Connector" (id 1) (at 28.575 55.88 0))
+    (property "Footprint" "Beirdo:QWIIC Connector" (id 2) (at 27.432 67.31 0)
       (effects (font (size 0.508 0.508)) hide)
     )
@@
     (in_bom yes) (on_board yes) (fields_autoplaced)
     (property "Reference" "J101" (id 0) (at 28.575 30.48 0))
-    (property "Value" "I2C_STANDARD" (id 1) (at 28.575 33.02 0))
-    (property "Footprint" "UltraLibrarian:PRT-16766" (id 2) (at 27.432 44.45 0)
+    (property "Value" "QWIIC Connector" (id 1) (at 28.575 33.02 0))
+    (property "Footprint" "Beirdo:QWIIC Connector" (id 2) (at 27.432 44.45 0)
       (effects (font (size 0.508 0.508)) hide)
     )
@@
     )
     (path "/2c528172-d77a-4cae-aaf4-a70b9bd06bda"
-      (reference "D101") (unit 1) (value "MMBZ27VALT116") (footprint "SparkFun-DiscreteSemi:SOT23-3")
+      (reference "D101") (unit 1) (value "MMBZ27VALT116") (footprint "SparkFun-Silicon-Standard:SOT23-3")
     )
     (path "/049af3e7-0792-4af9-989a-3d3cb3b7918f"
-      (reference "D102") (unit 1) (value "MMBZ27VALT116") (footprint "SparkFun-DiscreteSemi:SOT23-3")
+      (reference "D102") (unit 1) (value "MMBZ27VALT116") (footprint "SparkFun-Silicon-Standard:SOT23-3")
     )
     (path "/78cefd11-534c-468d-85be-e0507d57b0f6"
-      (reference "D103") (unit 1) (value "MMBZ27VCLT1") (footprint "SparkFun-DiscreteSemi:SOT23-3")
+      (reference "D103") (unit 1) (value "MMBZ27VCLT1") (footprint "SparkFun-Silicon-Standard:SOT23-3")
     )
     (path "/3e226555-24cf-4f93-b1fe-8eb6f44de7e8"
-      (reference "D104") (unit 1) (value "PESD1CAN") (footprint "SparkFun-DiscreteSemi:SOT23-3")
+      (reference "D104") (unit 1) (value "PESD1CAN") (footprint "SparkFun-Silicon-Standard:SOT23-3")
     )
     (path "/7e99a163-cc1f-415e-be4e-8ccc3d5be184"
-      (reference "D105") (unit 1) (value "PESD1CAN") (footprint "SparkFun-DiscreteSemi:SOT23-3")
+      (reference "D105") (unit 1) (value "PESD1CAN") (footprint "SparkFun-Silicon-Standard:SOT23-3")
     )
     (path "/2940c1f3-5f8f-4a77-b9a5-3db797a9d050/42280483-c97e-4e7f-b111-ccfb8c68e1a9"
@@
     )
     (path "/88611199-def1-4be6-a60e-948d7f3245f7"
-      (reference "J101") (unit 1) (value "I2C_STANDARD") (footprint "UltraLibrarian:PRT-16766")
+      (reference "J101") (unit 1) (value "QWIIC Connector") (footprint "Beirdo:QWIIC Connector")
     )
     (path "/0a47dc26-92e9-40e8-962d-6b9cd2b2309d"
@@
     )
     (path "/816bb22f-aaad-4066-9a31-e81a614b5655"
-      (reference "J103") (unit 1) (value "I2C_STANDARD") (footprint "UltraLibrarian:PRT-16766")
+      (reference "J103") (unit 1) (value "QWIIC Connector") (footprint "Beirdo:QWIIC Connector")
     )
     (path "/2940c1f3-5f8f-4a77-b9a5-3db797a9d050/e6a37936-27b5-4472-92d5-f4740dcb28dc"

Commit message: Switch out the PIC for an ATtiny424.
Parts:
- renumbered D105 to D1, D104 to D2, D103 to D3, D101 to D4, D102 to D5, J101 to J1, J103 to J2, J102 to J3
